Commit message: New robot model added

File: catkin_workspace/src/my_robot/urdf/my_robot_copy.xacro (robot description, xacro)
@@ -9,8 +9,8 @@
   </joint>
   <link name='chassis'>
-    <pose>0 0 0.2 0 0 0</pose>
+    <pose>0 0 0.1 0 0 0</pose>
     <inertial>
       <mass value="15.0"/>
-      <origin xyz="0 0 0" rpy=" 0 0 0"/>
+      <origin xyz="0.0 0 0" rpy=" 0 0 0"/>
       <inertia
           ixx="0.1" ixy="0" ixz="0"
@@ -20,35 +20,35 @@
     </inertial>
     <collision name='collision'>
-      <origin xyz="0 0 0" rpy=" 0 1.5707 0 "/>
-      <geometry>
-	 <cylinder length=".4" radius="0.1"/>
+      <origin xyz="0 0 0" rpy=" 0 0 0"/>
+      <geometry>
+        <box size=".4 .2 .1"/>
       </geometry>
     </collision>
     <visual name='chassis_visual'>
-      <origin xyz="0 0 0" rpy=" 0 1.5707 0 "/>
-      <geometry>
-	 <cylinder length=".4" radius="0.1"/>
+      <origin xyz="0 0 0" rpy=" 0 0 0"/>
+      <geometry>
+        <box size=".4 .2 .1"/>
       </geometry>
     </visual>
     <collision name='back_caster_collision'>
-      <origin xyz="-0.2 0 -0.1" rpy=" 0 0 0"/>
+      <origin xyz="-0.15 0 -0.05" rpy=" 0 0 0"/>
+      <geometry>
+        <sphere radius="0.0499"/>
+      </geometry>
+    </collision>
+    <visual name='back_caster_visual'>
+      <origin xyz="-0.15 0 -0.05" rpy=" 0 0 0"/>
       <geometry>
         <sphere radius="0.05"/>
       </geometry>
-    </collision>
-    <visual name='back_caster_visual'>
-      <origin xyz="-0.2 0 -0.1" rpy=" 0 0 0"/>
-      <geometry>
-        <sphere radius="0.05"/>
-      </geometry>
     </visual>
     <collision name='front_caster_collision'>
-      <origin xyz="0.2 0 -0.1" rpy=" 0 0 0"/>
-      <geometry>
-        <sphere radius="0.05"/>
+      <origin xyz="0.15 0 -0.05" rpy=" 0 0 0"/>
+      <geometry>
+        <sphere radius="0.0499"/>
       </geometry>
     </collision>
     <visual name='front_caster_visual'>
-      <origin xyz="0.2 0 -0.1" rpy=" 0 0 0"/>
+      <origin xyz="0.15 0 -0.05" rpy=" 0 0 0"/>
       <geometry>
         <sphere radius="0.05"/>
@@ -69,5 +69,5 @@
       <origin xyz="0 0 0" rpy=" 0 1.5707 1.5707"/>
       <geometry>
-	 <cylinder length="0.05" radius="0.2"/>
+	 <cylinder length="0.05" radius="0.1"/>
       </geometry>
     </collision>
@@ -75,5 +75,5 @@
       <origin xyz="0 0 0" rpy=" 0 1.5707 1.5707"/>
       <geometry>
-	 <cylinder length="0.05" radius="0.2"/>
+	 <cylinder length="0.05" radius="0.1"/>
       </geometry>
     </visual>
@@ -92,5 +92,5 @@
       <origin xyz="0 0 0" rpy=" 0 1.5707 1.5707"/>
       <geometry>
-	 <cylinder length="0.05" radius="0.2"/>
+	 <cylinder length="0.05" radius="0.1"/>
       </geometry>
     </collision>
@@ -98,10 +98,10 @@
       <origin xyz="0 0 0" rpy=" 0 1.5707 1.5707"/>
       <geometry>
-	 <cylinder length="0.05" radius="0.2"/>
+	 <cylinder length="0.05" radius="0.1"/>
       </geometry>
     </visual>
   </link>
  <joint type="continuous" name="left_wheel_hinge">
-    <origin xyz="0 0.2 0" rpy="0 0 0"/>
+    <origin xyz="0 0.15 0" rpy="0 0 0"/>
     <child link="left_wheel"/>
     <parent link="chassis"/>
@@ -112,5 +112,5 @@
   </joint>
   <joint type="continuous" name="right_wheel_hinge">
-    <origin xyz="0 -0.2 0" rpy="0 0 0"/>
+    <origin xyz="0 -0.15 0" rpy="0 0 0"/>
     <child link="right_wheel"/>
     <parent link="chassis"/>
@@ -186,32 +186,4 @@
     <dynamics damping="1.0" friction="1.0"/>
   </joint>
-<link name='cabin'>
-    <inertial>
-      <mass value=".5"/>
-      <origin xyz="0.0 0 0" rpy=" 0 0 0"/>
-      <inertia
-          ixx="0.05" ixy="0" ixz="0"
-          iyy="0.05" iyz="0"
-          izz="0.05"
-      />
-    </inertial>
-    <collision name='cabin_collision'>
-      <origin xyz="0 0 0" rpy=" 0 0 0"/>
-      <geometry>
-        <box size=".1 .2 .15"/>
-      </geometry>
-    </collision>y
-    <visual name='cabin_visual'>
-      <origin xyz="0 0 0" rpy=" 0 0 0 "/>
-      <geometry>
-        <box size=".1 .2 .15"/>
-      </geometry>
-    </visual>
-  </link>
-  <joint name="cabin_joint" type="fixed">
-    <origin xyz=" -.2 0 .05" rpy="0 0 0" />
-    <parent link="chassis"/>
-    <child link="cabin" />
-  </joint>
 <gazebo reference="left_wheel">
     <material>Gazebo/Green</material>
@@ -223,7 +195,4 @@
     <material>Gazebo/Blue</material>
 </gazebo>
-<gazebo reference="cabin">
-    <material>Gazebo/Blue</material>
-</gazebo>
 <gazebo reference="camera">
     <material>Gazebo/Red</material>
