Commit message: Ball chaser pkg added

File: catkin_ws/src/my_robot/urdf/my_robot.xacro (robot description, xacro)
@@ -1,4 +1,5 @@
 <?xml version='1.0'?>
 <robot name="my_robot" xmlns:xacro="http://www.ros.org/wiki/xacro">
+<xacro:include filename="$(find my_robot)/urdf/my_robot.gazebo" />
   <link name="robot_footprint"></link>
   <joint name="robot_footprint_joint" type="fixed">
@@ -108,4 +109,5 @@
     <limit effort="10000" velocity="1000"/>
     <dynamics damping="1.0" friction="1.0"/>
+    <commandTopic>cmd_vel</commandTopic>
   </joint>
   <joint type="continuous" name="right_wheel_hinge">
@@ -116,4 +118,5 @@
     <limit effort="10000" velocity="1000"/>
     <dynamics damping="1.0" friction="1.0"/>
+    <commandTopic>cmd_vel</commandTopic>
   </joint>
  <link name='camera'>
@@ -140,4 +143,5 @@
       </geometry>
     </visual>
+  <imageTopicName>rgb/image_raw</imageTopicName>
   </link>
   <joint type="fixed" name="camera_joint">
@@ -172,4 +176,5 @@
       </geometry>
     </visual>
+   <topicName>/scan</topicName>
   </link>
   <joint type="fixed" name="hokuyo_joint">
@@ -181,3 +186,18 @@
     <dynamics damping="1.0" friction="1.0"/>
   </joint>
+<gazebo reference="left_wheel">
+    <material>Gazebo/Green</material>
+</gazebo>
+<gazebo reference="right_wheel">
+    <material>Gazebo/Green</material>
+</gazebo>
+<gazebo reference="chassis">
+    <material>Gazebo/Blue</material>
+</gazebo>
+<gazebo reference="camera">
+    <material>Gazebo/Red</material>
+</gazebo>
+<gazebo reference="hokuyo">
+    <material>Gazebo/Black</material>
+</gazebo>
 </robot>

Commit message: New more stable robot added

File: catkin_ws/src/my_robot/urdf/my_robot.xacro (robot description, xacro)
@@ -22,5 +22,5 @@
       <origin xyz="0 0 0" rpy=" 0 1.5707 0 "/>
       <geometry>
-	 <cylinder length=".4" radius="0.1"/>
+	 <cylinder length=".2" radius="0.1"/>
       </geometry>
     </collision>
@@ -28,9 +28,9 @@
       <origin xyz="0 0 0" rpy=" 0 1.5707 0 "/>
       <geometry>
-	 <cylinder length=".4" radius="0.1"/>
+	 <cylinder length=".2" radius="0.1"/>
       </geometry>
     </visual>
     <collision name='back_caster_collision'>
-      <origin xyz="-0.2 0 -0.1" rpy=" 0 0 0"/>
+      <origin xyz="-0.1 0 -0.1" rpy=" 0 0 0"/>
       <geometry>
         <sphere radius="0.05"/>
@@ -38,5 +38,5 @@
     </collision>
     <visual name='back_caster_visual'>
-      <origin xyz="-0.2 0 -0.1" rpy=" 0 0 0"/>
+      <origin xyz="-0.1 0 -0.1" rpy=" 0 0 0"/>
       <geometry>
         <sphere radius="0.05"/>
@@ -44,5 +44,5 @@
     </visual>
     <collision name='front_caster_collision'>
-      <origin xyz="0.2 0 -0.1" rpy=" 0 0 0"/>
+      <origin xyz="0.1 0 -0.1" rpy=" 0 0 0"/>
       <geometry>
         <sphere radius="0.05"/>
@@ -50,5 +50,5 @@
     </collision>
     <visual name='front_caster_visual'>
-      <origin xyz="0.2 0 -0.1" rpy=" 0 0 0"/>
+      <origin xyz="0.1 0 -0.1" rpy=" 0 0 0"/>
       <geometry>
         <sphere radius="0.05"/>
@@ -69,5 +69,5 @@
       <origin xyz="0 0 0" rpy=" 0 1.5707 1.5707"/>
       <geometry>
-	 <cylinder length="0.05" radius="0.2"/>
+	 <cylinder length="0.05" radius="0.1"/>
       </geometry>
     </collision>
@@ -75,5 +75,5 @@
       <origin xyz="0 0 0" rpy=" 0 1.5707 1.5707"/>
       <geometry>
-	 <cylinder length="0.05" radius="0.2"/>
+	 <cylinder length="0.05" radius="0.1"/>
       </geometry>
     </visual>
@@ -92,5 +92,5 @@
       <origin xyz="0 0 0" rpy=" 0 1.5707 1.5707"/>
       <geometry>
-	 <cylinder length="0.05" radius="0.2"/>
+	 <cylinder length="0.05" radius="0.1"/>
       </geometry>
     </collision>
@@ -98,10 +98,10 @@
       <origin xyz="0 0 0" rpy=" 0 1.5707 1.5707"/>
       <geometry>
-	 <cylinder length="0.05" radius="0.2"/>
+	 <cylinder length="0.05" radius="0.1"/>
       </geometry>
     </visual>
   </link>
  <joint type="continuous" name="left_wheel_hinge">
-    <origin xyz="0 0.2 0" rpy="0 0 0"/>
+    <origin xyz="0 0.2 -.1" rpy="0 0 0"/>
     <child link="left_wheel"/>
     <parent link="chassis"/>
@@ -112,5 +112,5 @@
   </joint>
   <joint type="continuous" name="right_wheel_hinge">
-    <origin xyz="0 -0.2 0" rpy="0 0 0"/>
+    <origin xyz="0 -0.2 -.1" rpy="0 0 0"/>
     <child link="right_wheel"/>
     <parent link="chassis"/>
@@ -146,5 +146,5 @@
   </link>
   <joint type="fixed" name="camera_joint">
-    <origin xyz="0.2 0 0" rpy="0 0 0"/>
+    <origin xyz="0.1 0 0" rpy="0 0 0"/>
     <child link="camera"/>
     <parent link="chassis"/>
@@ -179,7 +179,7 @@
   </link>
   <joint type="fixed" name="hokuyo_joint">
-    <origin xyz="0.15 0 0.1" rpy="0 0 0"/>
+    <origin xyz="0 0 0.1" rpy="0 0 0"/>
     <child link="hokuyo"/>
-    <parent link="chassis"/>
+    <parent link="cabin"/>
     <axis xyz="0 1 0" rpy="0 0 0"/>
     <limit effort="10000" velocity="1000"/>
@@ -188,10 +188,10 @@
 <link name='cabin'>
     <inertial>
-      <mass value=".5"/>
-      <origin xyz="0.0 0 0" rpy=" 0 0 0"/>
-      <inertia
-          ixx="0.05" ixy="0" ixz="0"
-          iyy="0.05" iyz="0"
-          izz="0.05"
+      <mass value="0.0999"/>
+      <origin xyz="0.0 0 0" rpy=" 0 0 0"/>
+      <inertia
+          ixx="0.1" ixy="0" ixz="0"
+          iyy="0.1" iyz="0"
+          izz="0.1"
       />
     </inertial>
@@ -199,5 +199,5 @@
       <origin xyz="0 0 0" rpy=" 0 0 0"/>
       <geometry>
-        <box size=".1 .2 .15"/>
+        <box size=".1 .2 .2"/>
       </geometry>
     </collision>y
@@ -205,12 +205,40 @@
       <origin xyz="0 0 0" rpy=" 0 0 0 "/>
       <geometry>
-        <box size=".1 .2 .15"/>
+        <box size=".1 .2 .2"/>
       </geometry>
     </visual>
   </link>
   <joint name="cabin_joint" type="fixed">
-    <origin xyz=" -.2 0 .05" rpy="0 0 0" />
+    <origin xyz=" -.1 0 0" rpy="0 0 0" />
     <parent link="chassis"/>
     <child link="cabin" />
+  </joint>
+<link name='u_cabin'>
+    <inertial>
+      <mass value="1e-5"/>
+      <origin xyz="0.0 0 0" rpy=" 0 0 0"/>
+      <inertia
+          ixx="1e-6" ixy="0" ixz="0"
+          iyy="1e-6" iyz="0"
+          izz="1e-6"
+      />
+    </inertial>
+       <collision name='u_cabin_collision'>
+      <origin xyz="0 0 0" rpy=" 0 0 0"/>
+      <geometry>
+        <box size=".1 .1 .1"/>
+      </geometry>
+    </collision>
+    <visual name='u_cabin_visual'>
+      <origin xyz="0 0 0" rpy=" 0 0 0 "/>
+      <geometry>
+        <box size=".1 .1 .1"/>
+      </geometry>
+    </visual>
+  </link>
+  <joint name="u_cabin_joint" type="fixed">
+    <origin xyz=" 0 0 -.1" rpy="0 0 0" />
+    <parent link="cabin"/>
+    <child link="u_cabin" />
   </joint>
 <gazebo reference="left_wheel">

Commit message: Cylinder robot added

File: catkin_ws/src/my_robot/urdf/my_robot.xacro (robot description, xacro)
@@ -9,5 +9,5 @@
   </joint>
   <link name='chassis'>
-    <pose>0 0 0.2 0 0 0</pose>
+    <pose>0 0 0.1 0 0 0</pose>
     <inertial>
       <mass value="15.0"/>
@@ -20,37 +20,37 @@
     </inertial>
     <collision name='collision'>
-      <origin xyz="0 0 0" rpy=" 0 1.5707 0 "/>
-      <geometry>
-	 <cylinder length=".2" radius="0.1"/>
+      <origin xyz="0 0 0" rpy=" 0 0 0 "/>
+      <geometry>
+	 <cylinder length=".1" radius="0.2"/>
       </geometry>
     </collision>
     <visual name='chassis_visual'>
-      <origin xyz="0 0 0" rpy=" 0 1.5707 0 "/>
-      <geometry>
-	 <cylinder length=".2" radius="0.1"/>
+      <origin xyz="0 0 0" rpy=" 0 0 0 "/>
+      <geometry>
+	 <cylinder length=".1" radius="0.2"/>
       </geometry>
     </visual>
     <collision name='back_caster_collision'>
-      <origin xyz="-0.1 0 -0.1" rpy=" 0 0 0"/>
-      <geometry>
-        <sphere radius="0.05"/>
+      <origin xyz="-0.15 0 -0.1" rpy="1.5707 0 0"/>
+      <geometry>
+	 <cylinder length=".15" radius="0.0499"/>
       </geometry>
     </collision>
     <visual name='back_caster_visual'>
-      <origin xyz="-0.1 0 -0.1" rpy=" 0 0 0"/>
-      <geometry>
-        <sphere radius="0.05"/>
+      <origin xyz="-0.15 0 -0.1" rpy="1.5707 0 0 "/>
+      <geometry>
+	 <cylinder length=".15" radius="0.05"/>
       </geometry>
     </visual>
     <collision name='front_caster_collision'>
-      <origin xyz="0.1 0 -0.1" rpy=" 0 0 0"/>
-      <geometry>
-        <sphere radius="0.05"/>
+      <origin xyz="0.15 0 -0.1" rpy="1.5707 0 0 "/>
+      <geometry>
+	 <cylinder length=".15" radius="0.0499"/>
       </geometry>
     </collision>
     <visual name='front_caster_visual'>
-      <origin xyz="0.1 0 -0.1" rpy=" 0 0 0"/>
-      <geometry>
-        <sphere radius="0.05"/>
+      <origin xyz="0.15 0 -0.1" rpy="1.5707 0 0 "/>
+      <geometry>
+	 <cylinder length=".15" radius="0.05"/>
       </geometry>
     </visual>
@@ -103,5 +103,5 @@
   </link>
  <joint type="continuous" name="left_wheel_hinge">
-    <origin xyz="0 0.2 -.1" rpy="0 0 0"/>
+    <origin xyz="0 0.2 -.05" rpy="0 0 0"/>
     <child link="left_wheel"/>
     <parent link="chassis"/>
@@ -112,5 +112,5 @@
   </joint>
   <joint type="continuous" name="right_wheel_hinge">
-    <origin xyz="0 -0.2 -.1" rpy="0 0 0"/>
+    <origin xyz="0 -0.2 -.05" rpy="0 0 0"/>
     <child link="right_wheel"/>
     <parent link="chassis"/>
@@ -132,13 +132,13 @@
     </inertial>
      <collision name='camera_collision'>
-      <origin xyz="0 0 0" rpy=" 0 0 0"/>
-      <geometry>
-        <box size=".05 .05 .05"/>
+      <origin xyz="0 0 0" rpy=" 0 1.5707 0"/>
+      <geometry>
+	 <cylinder length="0.05" radius="0.05"/>
       </geometry>
     </collision>
     <visual name='camera_visual'>
-      <origin xyz="0 0 0" rpy=" 0 0 0"/>
-      <geometry>
-        <box size=".05 .05 .05"/>
+      <origin xyz="0 0 0" rpy=" 0 1.5707 0"/>
+      <geometry>
+	 <cylinder length="0.05" radius="0.05"/>
       </geometry>
     </visual>
@@ -146,5 +146,5 @@
   </link>
   <joint type="fixed" name="camera_joint">
-    <origin xyz="0.1 0 0" rpy="0 0 0"/>
+    <origin xyz="0.2 0 0" rpy="0 0 0"/>
     <child link="camera"/>
     <parent link="chassis"/>
@@ -179,5 +179,5 @@
   </link>
   <joint type="fixed" name="hokuyo_joint">
-    <origin xyz="0 0 0.1" rpy="0 0 0"/>
+    <origin xyz="0 0 0.05" rpy="0 0 0"/>
     <child link="hokuyo"/>
     <parent link="cabin"/>
@@ -188,10 +188,10 @@
 <link name='cabin'>
     <inertial>
-      <mass value="0.0999"/>
+      <mass value=".5"/>
       <origin xyz="0.0 0 0" rpy=" 0 0 0"/>
       <inertia
-          ixx="0.1" ixy="0" ixz="0"
-          iyy="0.1" iyz="0"
-          izz="0.1"
+          ixx="0.05" ixy="0" ixz="0"
+          iyy="0.05" iyz="0"
+          izz="0.05"
       />
     </inertial>
@@ -199,5 +199,5 @@
       <origin xyz="0 0 0" rpy=" 0 0 0"/>
       <geometry>
-        <box size=".1 .2 .2"/>
+        <box size=".2 .2 .1"/>
       </geometry>
     </collision>y
@@ -205,40 +205,12 @@
       <origin xyz="0 0 0" rpy=" 0 0 0 "/>
       <geometry>
-        <box size=".1 .2 .2"/>
+        <box size=".2 .2 .1"/>
       </geometry>
     </visual>
   </link>
   <joint name="cabin_joint" type="fixed">
-    <origin xyz=" -.1 0 0" rpy="0 0 0" />
+    <origin xyz=" 0 0 .05" rpy="0 0 0" />
     <parent link="chassis"/>
     <child link="cabin" />
-  </joint>
-<link name='u_cabin'>
-    <inertial>
-      <mass value="1e-5"/>
-      <origin xyz="0.0 0 0" rpy=" 0 0 0"/>
-      <inertia
-          ixx="1e-6" ixy="0" ixz="0"
-          iyy="1e-6" iyz="0"
-          izz="1e-6"
-      />
-    </inertial>
-       <collision name='u_cabin_collision'>
-      <origin xyz="0 0 0" rpy=" 0 0 0"/>
-      <geometry>
-        <box size=".1 .1 .1"/>
-      </geometry>
-    </collision>
-    <visual name='u_cabin_visual'>
-      <origin xyz="0 0 0" rpy=" 0 0 0 "/>
-      <geometry>
-        <box size=".1 .1 .1"/>
-      </geometry>
-    </visual>
-  </link>
-  <joint name="u_cabin_joint" type="fixed">
-    <origin xyz=" 0 0 -.1" rpy="0 0 0" />
-    <parent link="cabin"/>
-    <child link="u_cabin" />
   </joint>
 <gazebo reference="left_wheel">
@@ -252,5 +224,5 @@
 </gazebo>
 <gazebo reference="cabin">
-    <material>Gazebo/Blue</material>
+    <material>Gazebo/Yellow</material>
 </gazebo>
 <gazebo reference="camera">

Commit message: Project 4 done

File: catkin_ws/src/my_robot/urdf/my_robot.xacro (robot description, xacro)
@@ -179,5 +179,5 @@
   </link>
   <joint type="fixed" name="hokuyo_joint">
-    <origin xyz="0 0 0.05" rpy="0 0 0"/>
+    <origin xyz="0 0 0.1" rpy="0 0 0"/>
     <child link="hokuyo"/>
     <parent link="cabin"/>

Commit message: add rtabmap

File: catkin_ws/src/my_robot/urdf/my_robot.xacro (robot description, xacro)
@@ -209,4 +209,11 @@
     </visual>
   </link>
+  <joint name="camera_optical_joint" type="fixed">
+    <origin xyz="0 0 0" rpy="-1.5707 0 -1.5707"/>
+    <parent link="camera"/>
+    <child link="camera_optical"/>
+  </joint>
+  <link name="camera_optical">
+  </link>
   <joint name="cabin_joint" type="fixed">
     <origin xyz=" 0 0 .05" rpy="0 0 0" />
